Commit message: Maybe fixed the table and table macro stuff to work

File: Step2/table.urdf.xacro (robot description, xacro)
@@ -1,25 +1,13 @@
-<?xml version="1.0"?>
-<robot name="table" xmlns:xacro="http://www.ros.org/wiki/xacro">
-  <xacro:include filename="table_macro.xacro"/>
-  <!-- ================= PROPERTIES ================= -->
-  <xacro:property name="table_length" value="2"/>
-  <xacro:property name="table_width" value="1"/>
-  <xacro:property name="table_height" value="1"/>
-  <xacro:property name="table_thickness" value="0.05"/>
-  <xacro:property name="leg_length" value="${table_height - table_thickness}"/>
-  <xacro:property name="leg_radius" value="0.05"/>
-  <xacro:property name="prefix" value="table"/>
-  <xacro:property name="parent" value="world"/>
-  <!-- Instantiate table -->
-  <xacro:table
-      table_length="${table_length}"
-      table_width="${table_width}"
-      table_height="${table_height}"
-      table_thickness="${table_thickness}"
-      leg_length="${leg_length}"
-      leg_radius="${leg_radius}"
-      prefix="${prefix}"
-      parent="${parent}">
-    <origin xyz="0 0 1" rpy="0 0 0"/>
-  </xacro:table>
+<?xml version="1.0" encoding="UTF-8"?>
+<robot xmlns:xacro="http://wiki.ros.org/xacro" name="rrbot">
+  <!-- copy and paste the contents of "rrbot_macro.xacro" here -->
+  <xacro:include filename="materials.xacro" />
+  <xacro:include filename="table_macro.urdf.xacro"/>
+  <!-- create link fixed to the "world" -->
+  <link name="world" />
+  <!-- create the table and legs -->
+  <xacro:rrbot prefix="table" parent="world">
+    <!-- position table in the world -->
+    <origin xyz="0 0 1" rpy="0 0 0" />
+  </xacro:rrbot>
 </robot>

File: Step2/table_macro.xacro (robot description, xacro)
@@ -1,21 +1,12 @@
 <?xml version="1.0"?>
 <robot xmlns:xacro="http://www.ros.org/wiki/xacro">
-  <xacro:macro name="table" params="
-      table_length
-      table_width
-      table_height
-      table_thickness
-      leg_length
-      leg_radius
-      prefix
-      parent
-      *origin">
-    <!-- Materials -->
-    <material name="brown">
-      <color rgba="0.54 0.27 0.07 1.0"/>
-    </material>
-    <material name="light_grey">
-      <color rgba="0.8 0.8 0.8 1.0"/>
-    </material>
+  <xacro:macro name="table" params="prefix parent *origin">
+    <!-- ================= PROPERTIES ================= -->
+    <xacro:property name="table_length" value="2"/>
+    <xacro:property name="table_width" value="1"/>
+    <xacro:property name="table_height" value="1"/>
+    <xacro:property name="table_thickness" value="0.05"/>
+    <xacro:property name="leg_length" value="${table_height - table_thickness}"/>
+    <xacro:property name="leg_radius" value="0.05"/>
     <!-- ================= TABLE TOP ================= -->
     <!-- Frame at TOP surface -->
@@ -39,5 +30,5 @@
     <xacro:property name="leg_y" value="${table_width/2 - leg_radius}"/>
     <!-- ================= LEGS ================= -->
-    <xacro:macro name="leg" params="name x y">
+    <xacro:macro name="leg" params="prefix parent x y">
       <link name="${name}">
         <visual>
@@ -51,14 +42,14 @@
       </link>
       <joint name="table_to_${name}" type="fixed">
-        <parent link="table_top"/>
-        <child link="${name}"/>
+        <parent link="${parent}"/>
+        <child link="${prefix}"/>
         <origin xyz="${x} ${y} ${-table_thickness}" rpy="0 0 0"/>
       </joint>
     </xacro:macro>
     <!-- Instantiate four legs -->
-    <xacro:leg name="leg_fl" x="${leg_x}"  y="${leg_y}"/>
-    <xacro:leg name="leg_fr" x="${leg_x}"  y="${-leg_y}"/>
-    <xacro:leg name="leg_bl" x="${-leg_x}" y="${leg_y}"/>
-    <xacro:leg name="leg_br" x="${-leg_x}" y="${-leg_y}"/>
+    <xacro:leg prefix="leg_fl" parent="table" x="${leg_x}"  y="${leg_y}"/>
+    <xacro:leg prefix="leg_fr" parent="table" x="${leg_x}"  y="${-leg_y}"/>
+    <xacro:leg prefix="leg_bl" parent="table" x="${-leg_x}" y="${leg_y}"/>
+    <xacro:leg prefix="leg_br" parent="table" x="${-leg_x}" y="${-leg_y}"/>
   </xacro:macro>
 </robot>
