Commit message: Stuck on task2

File: Step2/rrbot_on_table.urdf.xacro (robot description, xacro)
@@ -5,8 +5,8 @@
     <xacro:include filename="rrbot_macro.xacro" />
     <link name="world" />
-    <xacro:table prefix="table_" parent="world">
+    <xacro:table prefix="table" parent="world">
         <origin xyz="0 0 1" rpy="0 0 0" />
     </xacro:table>
-    <xacro:rrbot prefix="rrbot_" parent="table_top">
+    <xacro:rrbot prefix="rrbot" parent="table_top">
         <origin xyz="0 0 0" rpy="0 0 0" />
     </xacro:rrbot>

File: Step2/table.urdf.xacro (robot description, xacro)
@@ -9,4 +9,6 @@
   <xacro:property name="leg_length" value="${table_height - table_thickness}"/>
   <xacro:property name="leg_radius" value="0.05"/>
+  <xacro:property name="prefix" value="table"/>
+  <xacro:property name="parent" value="world" />
   <!-- Instantiate table -->
   <xacro:table
@@ -16,4 +18,6 @@
       table_thickness="${table_thickness}"
       leg_length="${leg_length}"
-      leg_radius="${leg_radius}"/>
+      leg_radius="${leg_radius}"
+      prefix = "${prefix}"
+      parent = "${parent}" />
 </robot>

File: Step2/table_macro.xacro (robot description, xacro)
@@ -7,5 +7,7 @@
       table_thickness
       leg_length
-      leg_radius">
+      leg_radius
+      prefix
+      parent">
     <!-- Materials -->
     <material name="brown">
@@ -19,5 +21,5 @@
     <!-- ================= TABLE TOP ================= -->
     <!-- Frame at TOP surface -->
-    <link name="table_top">
+    <link name="${prefix}_top">
       <visual>
         <origin xyz="0 0 ${-table_thickness/2}" rpy="0 0 0"/>
@@ -29,5 +31,5 @@
     </link>
     <!-- World to table -->
-    <joint name="world_to_table" type="fixed">
+    <joint name="${parent}_to_${prefix}" type="fixed">
       <parent link="world"/>
       <child link="table_top"/>
@@ -52,5 +54,5 @@
         <parent link="table_top"/>
         <child link="${name}"/>
-        <origin xyz="${x} ${y} 0" rpy="0 0 0"/>
+        <origin xyz="${x} ${y} ${-table_thickness}" rpy="0 0 0"/>
       </joint>
     </xacro:macro>

Commit message: Still having trouble with step2 task2

File: Step2/rrbot_on_table.urdf.xacro (robot description, xacro)
@@ -5,5 +5,11 @@
     <xacro:include filename="rrbot_macro.xacro" />
     <link name="world" />
-    <xacro:table prefix="table" parent="world">
+    <xacro:table prefix="table" parent="world"
+        table_length="2"
+        table_width="1"
+        table_height="1"
+        table_thickness="0.05"
+        leg_length="0.95"
+        leg_radius="0.05">
         <origin xyz="0 0 1" rpy="0 0 0" />
     </xacro:table>

File: Step2/table.urdf.xacro (robot description, xacro)
@@ -10,5 +10,5 @@
   <xacro:property name="leg_radius" value="0.05"/>
   <xacro:property name="prefix" value="table"/>
-  <xacro:property name="parent" value="world" />
+  <xacro:property name="parent" value="world"/>
   <!-- Instantiate table -->
   <xacro:table
@@ -19,5 +19,7 @@
       leg_length="${leg_length}"
       leg_radius="${leg_radius}"
-      prefix = "${prefix}"
-      parent = "${parent}" />
+      prefix="${prefix}"
+      parent="${parent}">
+    <origin xyz="0 0 1" rpy="0 0 0"/>
+  </xacro:table>
 </robot>

File: Step2/table_macro.xacro (robot description, xacro)
@@ -9,5 +9,6 @@
       leg_radius
       prefix
-      parent">
+      parent
+      *origin">
     <!-- Materials -->
     <material name="brown">
@@ -17,6 +18,4 @@
       <color rgba="0.8 0.8 0.8 1.0"/>
     </material>
-    <!-- World -->
-    <link name="world"/>
     <!-- ================= TABLE TOP ================= -->
     <!-- Frame at TOP surface -->
@@ -32,7 +31,7 @@
     <!-- World to table -->
     <joint name="${parent}_to_${prefix}" type="fixed">
-      <parent link="world"/>
-      <child link="table_top"/>
-      <origin xyz="0 0 ${table_height}" rpy="0 0 0"/>
+      <parent link="${parent}"/>
+      <child link="${prefix}_top"/>
+      <xacro:insert_block name="origin"/>
     </joint>
     <!-- Compute leg offsets -->

Commit message: new changes to try to redo part 1

File: Step2/rrbot_on_table.urdf.xacro (robot description, xacro)
@@ -5,11 +5,5 @@
     <xacro:include filename="rrbot_macro.xacro" />
     <link name="world" />
-    <xacro:table prefix="table" parent="world"
-        table_length="2"
-        table_width="1"
-        table_height="1"
-        table_thickness="0.05"
-        leg_length="0.95"
-        leg_radius="0.05">
+    <xacro:table prefix="table" parent="world">
         <origin xyz="0 0 1" rpy="0 0 0" />
     </xacro:table>

File: Step2/table.urdf.xacro (robot description, xacro)
@@ -1,13 +1,9 @@
 <?xml version="1.0" encoding="UTF-8"?>
-<robot xmlns:xacro="http://wiki.ros.org/xacro" name="rrbot">
-  <!-- copy and paste the contents of "rrbot_macro.xacro" here -->
-  <xacro:include filename="materials.xacro" />
+<robot name="table" xmlns:xacro="http://wiki.ros.org/xacro">
+  <xacro:include filename="materials.xacro"/>
   <xacro:include filename="table_macro.urdf.xacro"/>
-  <!-- create link fixed to the "world" -->
-  <link name="world" />
-  <!-- create the table and legs -->
-  <xacro:rrbot prefix="table" parent="world">
-    <!-- position table in the world -->
-    <origin xyz="0 0 1" rpy="0 0 0" />
-  </xacro:rrbot>
+  <link name="world"/>
+  <xacro:table prefix="table" parent="world">
+    <origin xyz="0 0 1" rpy="0 0 0"/>
+  </xacro:table>
 </robot>

Commit message: Everything working, now problem with the robot's links being connected to the right frames

File: Step2/rrbot_on_table.urdf.xacro (robot description, xacro)
@@ -8,5 +8,5 @@
         <origin xyz="0 0 1" rpy="0 0 0" />
     </xacro:table>
-    <xacro:rrbot prefix="rrbot" parent="table_top">
+    <xacro:rrbot prefix="rrbot_" parent="table_top">
         <origin xyz="0 0 0" rpy="0 0 0" />
     </xacro:rrbot>

File: Step2/table.urdf.xacro (robot description, xacro)
@@ -2,5 +2,5 @@
 <robot name="table" xmlns:xacro="http://wiki.ros.org/xacro">
   <xacro:include filename="materials.xacro"/>
-  <xacro:include filename="table_macro.urdf.xacro"/>
+  <xacro:include filename="table_macro.xacro"/>
   <link name="world"/>
   <xacro:table prefix="table" parent="world">

File: Step2/table_macro.xacro (robot description, xacro)
@@ -1,3 +1,4 @@
 <?xml version="1.0"?>
+<robot xmlns:xacro="http://www.ros.org/wiki/xacro">
   <xacro:macro name="table" params="prefix parent *origin">
     <!-- ================= PROPERTIES ================= -->
@@ -8,4 +9,10 @@
     <xacro:property name="leg_length" value="${table_height - table_thickness}"/>
     <xacro:property name="leg_radius" value="0.05"/>
+    <!-- World to table -->
+    <joint name="${prefix}_to_${parent}" type="fixed">
+      <xacro:insert_block name="origin"/>
+      <parent link="${parent}"/>
+      <child link="${prefix}_top"/>
+    </joint>
     <!-- ================= TABLE TOP ================= -->
     <!-- Frame at TOP surface -->
@@ -19,16 +26,10 @@
       </visual>
     </link>
-    <!-- World to table -->
-    <joint name="${parent}_to_${prefix}" type="fixed">
-      <parent link="${parent}"/>
-      <child link="${prefix}_top"/>
-      <xacro:insert_block name="origin"/>
-    </joint>
     <!-- Compute leg offsets -->
     <xacro:property name="leg_x" value="${table_length/2 - leg_radius}"/>
     <xacro:property name="leg_y" value="${table_width/2 - leg_radius}"/>
     <!-- ================= LEGS ================= -->
-    <xacro:macro name="leg" params="prefix parent x y">
-      <link name="${prefix}">
+    <xacro:macro name="leg" params="name x y">
+      <link name="${name}">
         <visual>
           <!-- Frame at TOP of leg -->
@@ -40,14 +41,15 @@
         </visual>
       </link>
-      <joint name="table_to_${prefix}" type="fixed">
-        <parent link="${parent}"/>
-        <child link="${prefix}"/>
+      <joint name="table_to_${name}" type="fixed">
         <origin xyz="${x} ${y} ${-table_thickness}" rpy="0 0 0"/>
+        <parent link="table_top"/>
+        <child link="${name}"/>
       </joint>
     </xacro:macro>
     <!-- Instantiate four legs -->
-    <xacro:leg prefix="leg_fl" parent="table" x="${leg_x}"  y="${leg_y}"/>
-    <xacro:leg prefix="leg_fr" parent="table" x="${leg_x}"  y="${-leg_y}"/>
-    <xacro:leg prefix="leg_bl" parent="table" x="${-leg_x}" y="${leg_y}"/>
-    <xacro:leg prefix="leg_br" parent="table" x="${-leg_x}" y="${-leg_y}"/>
+    <xacro:leg name="leg_fl" x="${leg_x}"  y="${leg_y}"/>
+    <xacro:leg name="leg_fr" x="${leg_x}"  y="${-leg_y}"/>
+    <xacro:leg name="leg_bl" x="${-leg_x}" y="${leg_y}"/>
+    <xacro:leg name="leg_br" x="${-leg_x}" y="${-leg_y}"/>
   </xacro:macro>
+</robot>
