Commit message: Removed robot wrapper from table macro

File: Step2/table_macro.xacro (robot description, xacro)
@@ -1,4 +1,3 @@
 <?xml version="1.0"?>
-<robot xmlns:xacro="http://www.ros.org/wiki/xacro">
   <xacro:macro name="table" params="prefix parent *origin">
     <!-- ================= PROPERTIES ================= -->
@@ -31,5 +30,5 @@
     <!-- ================= LEGS ================= -->
     <xacro:macro name="leg" params="prefix parent x y">
-      <link name="${name}">
+      <link name="${prefix}">
         <visual>
           <!-- Frame at TOP of leg -->
@@ -41,5 +40,5 @@
         </visual>
       </link>
-      <joint name="table_to_${name}" type="fixed">
+      <joint name="table_to_${prefix}" type="fixed">
         <parent link="${parent}"/>
         <child link="${prefix}"/>
@@ -53,3 +52,2 @@
     <xacro:leg prefix="leg_br" parent="table" x="${-leg_x}" y="${-leg_y}"/>
   </xacro:macro>
-</robot>

Commit message: Working up to Task 4. Going to work on Task 4 on vscode on the mac instead of the remote pc

File: Step2/table_macro.xacro (robot description, xacro)
@@ -30,5 +30,5 @@
     <xacro:property name="leg_y" value="${table_width/2 - leg_radius}"/>
     <!-- ================= LEGS ================= -->
-    <xacro:macro name="leg" params="name x y">
+    <xacro:macro name="leg" params="name prefix x y">
       <link name="${name}">
         <visual>
@@ -41,15 +41,15 @@
         </visual>
       </link>
-      <joint name="table_to_${name}" type="fixed">
+      <joint name="${prefix}_to_${name}" type="fixed">
         <origin xyz="${x} ${y} ${-table_thickness}" rpy="0 0 0"/>
-        <parent link="table_top"/>
+        <parent link="${prefix}_top"/>
         <child link="${name}"/>
       </joint>
     </xacro:macro>
     <!-- Instantiate four legs -->
-    <xacro:leg name="leg_fl" x="${leg_x}"  y="${leg_y}"/>
-    <xacro:leg name="leg_fr" x="${leg_x}"  y="${-leg_y}"/>
-    <xacro:leg name="leg_bl" x="${-leg_x}" y="${leg_y}"/>
-    <xacro:leg name="leg_br" x="${-leg_x}" y="${-leg_y}"/>
+    <xacro:leg name="leg_fl" prefix="table" x="${leg_x}"  y="${leg_y}"/>
+    <xacro:leg name="leg_fr" prefix="table" x="${leg_x}"  y="${-leg_y}"/>
+    <xacro:leg name="leg_bl" prefix="table" x="${-leg_x}" y="${leg_y}"/>
+    <xacro:leg name="leg_br" prefix="table" x="${-leg_x}" y="${-leg_y}"/>
   </xacro:macro>
 </robot>

File: Step2/table_on_rrbot.urdf.xacro (robot description, xacro)
@@ -8,5 +8,5 @@
         <origin xyz="0 0 0" rpy="0 0 0" />
     </xacro:rrbot>
-    <xacro:table prefix="table_" parent="rrbot_tool0">
+    <xacro:table prefix="table" parent="rrbot_tool0">
         <origin xyz="0 0 0" rpy="${pi} 0 0" />
     </xacro:table>
