Commit message: Step2 Complete

File: Step2/robot_lab.urdf.xacro (robot description, xacro)
@@ -11,5 +11,5 @@
         <origin xyz="0 0 0" rpy="0 0 0" />
     </xacro:rrbot>
-        <xacro:table prefix="table2" parent="world">
+    <xacro:table prefix="table2" parent="world">
         <origin xyz="0 0 1" rpy="0 0 0" />
     </xacro:table>
@@ -17,5 +17,5 @@
         <origin xyz="0 0 0" rpy="0 0 0" />
     </xacro:rrbot>
-        <xacro:table prefix="table3" parent="world">
+    <xacro:table prefix="table3" parent="world">
         <origin xyz="3 0 1" rpy="0 0 0" />
     </xacro:table>
@@ -23,3 +23,21 @@
         <origin xyz="0 0 0" rpy="0 0 0" />
     </xacro:rrbot>
+    <xacro:table prefix="table4" parent="world">
+        <origin xyz="-3 3 1" rpy="0 0 0" />
+    </xacro:table>
+    <xacro:rrbot prefix="rrbot4_" parent="table4_top">
+        <origin xyz="0 0 0" rpy="0 0 0" />
+    </xacro:rrbot>
+    <xacro:table prefix="table5" parent="world">
+        <origin xyz="0 3 1" rpy="0 0 0" />
+    </xacro:table>
+    <xacro:rrbot prefix="rrbot5_" parent="table5_top">
+        <origin xyz="0 0 0" rpy="0 0 0" />
+    </xacro:rrbot>
+        <xacro:table prefix="table6" parent="world">
+        <origin xyz="3 3 1" rpy="0 0 0" />
+    </xacro:table>
+    <xacro:rrbot prefix="rrbot6_" parent="table6_top">
+        <origin xyz="0 0 0" rpy="0 0 0" />
+    </xacro:rrbot>
 </robot>

File: Step2/table_macro.xacro (robot description, xacro)
@@ -48,8 +48,8 @@
     </xacro:macro>
     <!-- Instantiate four legs -->
-    <xacro:leg name="leg_fl" prefix="${prefix}" x="${leg_x}"  y="${leg_y}"/>
-    <xacro:leg name="leg_fr" prefix="${prefix}" x="${leg_x}"  y="${-leg_y}"/>
-    <xacro:leg name="leg_bl" prefix="${prefix}" x="${-leg_x}" y="${leg_y}"/>
-    <xacro:leg name="leg_br" prefix="${prefix}" x="${-leg_x}" y="${-leg_y}"/>
+    <xacro:leg name="${prefix}_leg_fl" prefix="${prefix}" x="${leg_x}"  y="${leg_y}"/>
+    <xacro:leg name="${prefix}_leg_fr" prefix="${prefix}" x="${leg_x}"  y="${-leg_y}"/>
+    <xacro:leg name="${prefix}_leg_bl" prefix="${prefix}" x="${-leg_x}" y="${leg_y}"/>
+    <xacro:leg name="${prefix}_leg_br" prefix="${prefix}" x="${-leg_x}" y="${-leg_y}"/>
   </xacro:macro>
 </robot>
